Commit message: Add Orbbec rough terrain project updates

File: src/get_urdf/model/simple_car.urdf (robot description, URDF)
Before this commit: robot simple_car, 7 links, 6 joints
Links:
- added link orbbec_front_depth_optical_frame
- added link orbbec_front_link, mass 0.12; collision box size=0.09 0.025 0.025; visual box size=0.09 0.025 0.025
- added link orbbec_rear_depth_optical_frame
- added link orbbec_rear_link, mass 0.12; collision box size=0.09 0.025 0.025; visual box size=0.09 0.025 0.025
Joints:
- added joint orbbec_front_depth_optical_joint: type fixed, parent orbbec_front_link, child orbbec_front_depth_optical_frame, origin xyz=0 0 0 rpy=0 0 0
- added joint orbbec_front_joint: type fixed, parent chassis, child orbbec_front_link, origin xyz=0.32 0 0.35 rpy=0 0.52 0
- added joint orbbec_rear_depth_optical_joint: type fixed, parent orbbec_rear_link, child orbbec_rear_depth_optical_frame, origin xyz=0 0 0 rpy=0 0 0
- added joint orbbec_rear_joint: type fixed, parent chassis, child orbbec_rear_link, origin xyz=-0.32 0 0.35 rpy=0 0.52 3.14159
